File: DoneByCoffee/SSOP20toSOIC20/SSOPtoSOIC.kicad_pcb (KiCad board)
At the start: 2 copper layers, 21.5 x 25.9 mm, 164 parts

Commit message: opa diff mode jobs
Parts:
- renumbered SSOP20 to DD1, SSOP20 to DD2, SSOP21 to DD3, SSOP22 to DD4
Other:
- board text added: "SSOP20 to SOIC20"
- board text removed: "to SOIC20"
