File: OpAmps/OpAmpOnDiffModePCB/OPADiffMode.kicad_sch (KiCad schematic)
At the start: 14 parts, among them J1 Screw_Terminal_01x11, J2 Conn_01x15

Commit message: opa diff mode jobs
Connections:
- net VBIAS1/VDD is gone; now on net VDA: J2.12 (Pin_12), R1.1
- net GNDD: no longer J1.1 (Pin_1), J1.11 (Pin_11), J1.6 (Pin_6)
- net AI4+: now reaches J1.3 (Pin_3)
- net AI3-: now reaches J1.4 (Pin_4)
- net VDA: now reaches J1.7 (Pin_7)
- net AI2+: now reaches J1.9 (Pin_9)
- net VEE: now reaches J2.10 (Pin_10), J2.13 (Pin_13), R3.1
- net VEE: now also J1.6 (Pin_6)
- net AI1 renamed AI4-
- net AI2 renamed AI3+
- net AI3 renamed AI2-
- net AI4 renamed AI1-
- net OPA1GND renamed GNDA
- new net AI1+: J1.11 (Pin_11)
- no-connect marks 4 -> 7
Other:
- sheet DiffMode1 ports: added ANInput, APInput; removed AInput
- moved on the sheet: J1, R1, R2, R3, R4
